Commit message: adding camera

File: urdf/so101.urdf (robot description, URDF)
Before this commit: robot so101_new_calib, 8 links, 7 joints
Links:
- added link d435i_link, mass 0.3592826634307687; collision mesh filename=package://so101_description/meshes/d435i.stl scale=0.001 0.001 0.001; visual mesh filename=package://so101_description/meshes/d435i.stl scale=0.001 0.001 0.001
- link gripper_link: geometry collision mesh filename=package://so101_description/meshes/jaw.stl scale=0.001 0.001 0.001; collision mesh filename=package://so101_description/meshes/sts3215_03a_v1.stl
- link moving_jaw_so101_v1_link: geometry collision mesh filename=package://so101_description/meshes/moving_jaw.stl scale=0.001 0.001 0.001; visual mesh filename=package://so101_description/meshes/moving_jaw.stl scale=0.001 0.001 0.001
Joints:
- added joint gripper_to_d435i: type fixed, parent gripper_link, child d435i_link, origin xyz=-0.02250293 0.05580957 -0.0140886 rpy=1.2217304763960246 -0.0000026535898 1.5707963267948966
